Commit message: Add 2step shelf

File: urdf/short_shelf_description.urdf.xacro (robot description, xacro)
@@ -41,22 +41,4 @@
     </collision>
   </link>
-  <!-- Top Plate Link -->
-  <link name="shelf_top_plate_link">
-    <visual>
-      <geometry>
-        <mesh filename="package://kachaka_shelf_description/stl/kachaka_shelf_plate.stl"/> <!-- PlateのSTLファイル -->
-      </geometry>
-       <material name="gray_material">
-        <color rgba="${gray}"/>
-      </material>
-      <origin xyz="-0.13 0 -${shelf_distance_short + 0.1}" rpy="0 0 1.5708"/>
-    </visual>
-    <collision>
-      <geometry>
-        <mesh filename="package://kachaka_shelf_description/stl/kachaka_shelf_plate.stl"/> <!-- PlateのSTLファイル -->
-      </geometry>
-      <origin xyz="-0.13 0 -${shelf_distance_short + 0.1}" rpy="0 0 1.5708"/>
-    </collision>
-  </link>
   <!-- Joint between Base and Middle Plate -->
   <joint name="base_to_middle" type="fixed">

Commit message: modifired model

File: urdf/short_shelf_description.urdf.xacro (robot description, xacro)
@@ -9,5 +9,5 @@
     <visual>
       <geometry>
-        <mesh filename="package://kachaka_shelf_description/stl/kachaka_shelf_base.stl"/> <!-- BaseのSTLファイル -->
+        <mesh filename="package://kachaka_shelf_description/stl/kachaka_shelf.stl" scale="0.001 0.001 0.001"/> <!-- BaseのSTLファイル -->
       </geometry>
       <material name="gray_material">
@@ -18,5 +18,5 @@
     <collision>
       <geometry>
-        <mesh filename="package://kachaka_shelf_description/stl/kachaka_shelf_base.stl"/> <!-- BaseのSTLファイル -->
+        <mesh filename="package://kachaka_shelf_description/stl/kachaka_shelf.stl" scale="0.001 0.001 0.001"/> <!-- BaseのSTLファイル -->
       </geometry>
       <origin xyz="-0.13 0 0" rpy="0 0 1.5708"/>
@@ -27,16 +27,18 @@
     <visual>
       <geometry>
-        <mesh filename="package://kachaka_shelf_description/stl/kachaka_shelf_plate.stl"/> <!-- PlateのSTLファイル -->
+        <mesh filename="package://kachaka_shelf_description/stl/kachaka_shelf.stl" scale="0.001 0.001 0.001"/> <!-- PlateのSTLファイル -->
       </geometry>
        <material name="gray_material">
         <color rgba="${gray}"/>
       </material>
-      <origin xyz="-0.13 0 -${shelf_distance_long}" rpy="0 0 1.5708"/>
+      <!-- origin xyz="-0.13 0 -${shelf_distance_long}" rpy="0 0 1.5708"/ -->
+      <origin xyz="-0.13 0 0" rpy="0 0 1.5708"/>
     </visual>
     <collision>
       <geometry>
-        <mesh filename="package://kachaka_shelf_description/stl/kachaka_shelf_plate.stl"/> <!-- PlateのSTLファイル -->
+        <mesh filename="package://kachaka_shelf_description/stl/kachaka_shelf.stl" scale="0.001 0.001 0.001"/> <!-- PlateのSTLファイル -->
       </geometry>
-      <origin xyz="-0.13 0 -${shelf_distance_long}" rpy="0 0 1.5708"/>
+      <!--origin xyz="-0.13 0 -${shelf_distance_long}" rpy="0 0 1.5708"/-->
+      <origin xyz="-0.13 0 0" rpy="0 0 1.5708"/>
     </collision>
   </link>
