Commit message: update

File: urdf/shelf_description.urdf.xacro (robot description, xacro)
@@ -9,5 +9,5 @@
     <visual>
       <geometry>
-        <mesh filename="package://kachaka_shelf_description/stl/kachaka_shelf_base.stl"/> <!-- BaseのSTLファイル -->
+        <mesh filename="package://kachaka_shelf_description/stl/kachaka_shelf.stl" scale="0.001 0.001 0.001"/> <!-- BaseのSTLファイル -->
       </geometry>
       <material name="gray_material">
@@ -18,5 +18,5 @@
     <collision>
       <geometry>
-        <mesh filename="package://kachaka_shelf_description/stl/kachaka_shelf_base.stl"/> <!-- BaseのSTLファイル -->
+        <mesh filename="package://kachaka_shelf_description/stl/kachaka_shelf.stl" scale="0.001 0.001 0.001"/> <!-- BaseのSTLファイル -->
       </geometry>
       <origin xyz="-0.13 0 0" rpy="0 0 1.5708"/>
@@ -27,16 +27,18 @@
     <visual>
       <geometry>
-        <mesh filename="package://kachaka_shelf_description/stl/kachaka_shelf_plate.stl"/> <!-- PlateのSTLファイル -->
+        <mesh filename="package://kachaka_shelf_description/stl/kachaka_shelf.stl" scale="0.001 0.001 0.001"/> <!-- PlateのSTLファイル -->
       </geometry>
        <material name="gray_material">
         <color rgba="${gray}"/>
       </material>
-      <origin xyz="-0.13 0 -${shelf_distance_long}" rpy="0 0 1.5708"/>
+      <!-- origin xyz="-0.13 0 -${shelf_distance_long}" rpy="0 0 1.5708"/ -->
+      <origin xyz="-0.13 0 0" rpy="0 0 1.5708"/>
     </visual>
     <collision>
       <geometry>
-        <mesh filename="package://kachaka_shelf_description/stl/kachaka_shelf_plate.stl"/> <!-- PlateのSTLファイル -->
+        <mesh filename="package://kachaka_shelf_description/stl/kachaka_shelf.stl" scale="0.001 0.001 0.001"/> <!-- PlateのSTLファイル -->
       </geometry>
-      <origin xyz="-0.13 0 -${shelf_distance_long}" rpy="0 0 1.5708"/>
+      <!--origin xyz="-0.13 0 -${shelf_distance_long}" rpy="0 0 1.5708"/-->
+      <origin xyz="-0.13 0 0" rpy="0 0 1.5708"/>
     </collision>
   </link>
@@ -45,16 +47,18 @@
     <visual>
       <geometry>
-        <mesh filename="package://kachaka_shelf_description/stl/kachaka_shelf_plate.stl"/> <!-- PlateのSTLファイル -->
+        <mesh filename="package://kachaka_shelf_description/stl/kachaka_shelf.stl" scale="0.001 0.001 0.001"/> <!-- PlateのSTLファイル -->
       </geometry>
        <material name="gray_material">
         <color rgba="${gray}"/>
       </material>
-      <origin xyz="-0.13 0 -${shelf_distance_short + 0.1}" rpy="0 0 1.5708"/>
+      <!-- origin xyz="-0.13 0 -${shelf_distance_long}" rpy="0 0 1.5708"/ -->
+      <origin xyz="-0.13 0 0" rpy="0 0 1.5708"/>
     </visual>
     <collision>
       <geometry>
-        <mesh filename="package://kachaka_shelf_description/stl/kachaka_shelf_plate.stl"/> <!-- PlateのSTLファイル -->
+        <mesh filename="package://kachaka_shelf_description/stl/kachaka_shelf.stl" scale="0.001 0.001 0.001"/> <!-- PlateのSTLファイル -->
       </geometry>
-      <origin xyz="-0.13 0 -${shelf_distance_short + 0.1}" rpy="0 0 1.5708"/>
+      <!--origin xyz="-0.13 0 -${shelf_distance_long}" rpy="0 0 1.5708"/-->
+      <origin xyz="-0.13 0 0" rpy="0 0 1.5708"/>
     </collision>
   </link>
@@ -63,7 +67,7 @@
     <parent link="shelf_base_link"/>
     <child link="shelf_middle_plate_link"/>
-    <origin xyz="0 0 ${shelf_distance_long}"/> <!-- Z軸方向に0.15m上 -->
+    <origin xyz="0 0 ${shelf_distance_short}"/> <!-- Z軸方向に0.15m上 -->
   </joint>
-  <!-- Joint between Middle Plate and Top Plate -->
+  <!-- Joint between Middle and Top Plate -->
   <joint name="middle_to_top" type="fixed">
     <parent link="shelf_middle_plate_link"/>
